File: DAC.kicad_sch (KiCad schematic)
At the start: 1 part, among them J3 165MDAC

Commit message: change logick
на платі будуть роз'єми, цап ацп підключаються плоским кабелем
Parts:
- J3: footprint pcbDAC:165M_DAC -> Connector_PinHeader_2.54mm:PinHeader_2x10_P2.54mm_Vertical
Changed lines of the file:
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@@
 			)
 		)
-		(property "Footprint" "pcbDAC:165M_DAC"
+		(property "Footprint" "Connector_PinHeader_2.54mm:PinHeader_2x10_P2.54mm_Vertical"
 			(at 106.68 76.2 0)
 			(effects

Commit message: Make 3d model for ADC and FPGA. Trying to assembly
Parts:
- J3: footprint Connector_PinHeader_2.54mm:PinHeader_2x10_P2.54mm_Vertical -> Library:CONN-TH_DS1011-20RBSIB7-B
Changed lines of the file:
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@@
 			)
 		)
-		(property "Footprint" "Connector_PinHeader_2.54mm:PinHeader_2x10_P2.54mm_Vertical"
+		(property "Footprint" "Library:CONN-TH_DS1011-20RBSIB7-B"
 			(at 106.68 76.2 0)
 			(effects
