File: adc.kicad_sch (KiCad schematic)
At the start: 1 part, among them J4 65MADC

Commit message: change logick
на платі будуть роз'єми, цап ацп підключаються плоским кабелем
Parts:
- J4: footprint pcbDAC:65M_ADC -> Connector_PinHeader_2.54mm:PinHeader_2x10_P2.54mm_Vertical
Changed lines of the file:
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@@
 			)
 		)
-		(property "Footprint" "pcbDAC:65M_ADC"
+		(property "Footprint" "Connector_PinHeader_2.54mm:PinHeader_2x10_P2.54mm_Vertical"
 			(at 99.06 71.12 0)
 			(effects

Commit message: Make 3d model for ADC and FPGA. Trying to assembly
Parts:
- J4: footprint Connector_PinHeader_2.54mm:PinHeader_2x10_P2.54mm_Vertical -> Library:CONN-TH_DS1011-20RBSIB7-B
Changed lines of the file:
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@@
-					(unit 1)
-				)
-				(path "/7e985ab5-4049-4d72-94c7-921d31b1011c/cdb974c5-a411-4323-b4cc-287c4c078a52"
-					(reference "#PWR032")
 					(unit 1)
 				)
@@
 					(unit 1)
 				)
-				(path "/7e985ab5-4049-4d72-94c7-921d31b1011c/cdb974c5-a411-4323-b4cc-287c4c078a52"
-					(reference "#PWR029")
-					(unit 1)
-				)
 			)
 		)
@@
 					(unit 1)
 				)
-				(path "/7e985ab5-4049-4d72-94c7-921d31b1011c/cdb974c5-a411-4323-b4cc-287c4c078a52"
-					(reference "#PWR028")
-					(unit 1)
-				)
 			)
 		)
@@
 				(path "/7e985ab5-4049-4d72-94c7-921d31b1011c/c44eb6c4-0c79-431d-b3ea-fcb1cd71cbdb"
 					(reference "#PWR021")
-					(unit 1)
-				)
-				(path "/7e985ab5-4049-4d72-94c7-921d31b1011c/cdb974c5-a411-4323-b4cc-287c4c078a52"
-					(reference "#PWR027")
 					(unit 1)
 				)
@@
 					(unit 1)
 				)
-				(path "/7e985ab5-4049-4d72-94c7-921d31b1011c/cdb974c5-a411-4323-b4cc-287c4c078a52"
-					(reference "#PWR031")
-					(unit 1)
-				)
 			)
 		)
@@
 			)
 		)
-		(property "Footprint" "Connector_PinHeader_2.54mm:PinHeader_2x10_P2.54mm_Vertical"
+		(property "Footprint" "Library:CONN-TH_DS1011-20RBSIB7-B"
 			(at 99.06 71.12 0)
 			(effects
@@
 					(unit 1)
 				)
-				(path "/7e985ab5-4049-4d72-94c7-921d31b1011c/cdb974c5-a411-4323-b4cc-287c4c078a52"
-					(reference "J5")
-					(unit 1)
-				)
 			)
 		)
@@
 					(unit 1)
 				)
-				(path "/7e985ab5-4049-4d72-94c7-921d31b1011c/cdb974c5-a411-4323-b4cc-287c4c078a52"
-					(reference "#PWR030")
-					(unit 1)
-				)
